File: MCU.kicad_sch (KiCad schematic)
At the start: 4 parts, among them U2 BL652

Commit message: updates from call
Parts:
- added J1: Conn_ARM_SWD_TagConnect_TC2030, Connector:Tag-Connect_TC2030-IDC-NL_2x03_P1.27mm_Vertical, symbol Connector:Conn_ARM_SWD_TagConnect_TC2030
Connections:
- net +3V3: now also J1.1 (VCC)
- net Audio_FIL: now also U2.21 (SIO_04/AIN2); no longer U2.23 (SIO_02/AIN0)
- net GND: now also J1.5 (GND)
- net SCL: no longer U2.6 (SWDCLK)
- net SDA: no longer U2.5 (SWDIO)
- net at R1.2, R2.1: now also U2.35 (SIO_28/AIN4); no longer U2.37 (SIO_26)
- new net SWCLK: J1.4 (SWCLK), U2.6 (SWDCLK)
- new net SWD: J1.2 (SWDIO), U2.5 (SWDIO)
Changed lines of the file:
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@@
+    (stroke (width 0) (type default))
+  )
+  (wire (pts (xy 154.94 80.01) (xy 160.02 80.01))
+    (stroke (width 0) (type default))
+  )
+  (wire (pts (xy 190.5 50.8) (xy 196.85 50.8))
     (stroke (width 0) (type default))
   )
@@
     (stroke (width 0) (type default))
   )
+  (wire (pts (xy 190.5 53.34) (xy 196.85 53.34))
+    (stroke (width 0) (type default))
+  )
+  (wire (pts (xy 154.94 82.55) (xy 160.02 82.55))
+    (stroke (width 0) (type default))
+  )
+  (wire (pts (xy 154.94 97.79) (xy 179.07 97.79))
+    (stroke (width 0) (type default))
+  )
   (wire (pts (xy 101.6 105.41) (xy 104.14 105.41))
     (stroke (width 0) (type default))
   )
-  (wire (pts (xy 179.07 90.17) (xy 179.07 102.87))
+  (wire (pts (xy 179.07 90.17) (xy 179.07 97.79))
     (stroke (width 0) (type default))
   )
@@
   )
   (wire (pts (xy 184.15 82.55) (xy 190.5 82.55))
-    (stroke (width 0) (type default))
-  )
-  (wire (pts (xy 179.07 102.87) (xy 154.94 102.87))
     (stroke (width 0) (type default))
   )
@@
     (effects (font (size 1.27 1.27)) (justify left bottom))
   )
+  (label "SWD" (at 193.04 53.34 0) (fields_autoplaced)
+    (effects (font (size 1.27 1.27)) (justify left bottom))
+  )
   (label "RES2" (at 101.6 105.41 0) (fields_autoplaced)
     (effects (font (size 1.27 1.27)) (justify left bottom))
   )
+  (label "SWD" (at 156.21 82.55 0) (fields_autoplaced)
+    (effects (font (size 1.27 1.27)) (justify left bottom))
+  )
+  (label "SWCLK" (at 156.21 80.01 0) (fields_autoplaced)
+    (effects (font (size 1.27 1.27)) (justify left bottom))
+  )
+  (label "SWCLK" (at 191.77 50.8 0) (fields_autoplaced)
+    (effects (font (size 1.27 1.27)) (justify left bottom))
+  )
   (label "RES" (at 101.6 102.87 0) (fields_autoplaced)
     (effects (font (size 1.27 1.27)) (justify left bottom))
@@
     (effects (font (size 1.27 1.27)) (justify right))
   )
-  (hierarchical_label "SDA" (shape output) (at 154.94 82.55 0) (fields_autoplaced)
+  (hierarchical_label "SDA" (shape output) (at 180.34 106.68 0) (fields_autoplaced)
     (effects (font (size 1.27 1.27)) (justify left))
   )
@@
     (effects (font (size 1.27 1.27)) (justify left))
   )
-  (hierarchical_label "Audio_FIL" (shape input) (at 104.14 85.09 180) (fields_autoplaced)
-    (effects (font (size 1.27 1.27)) (justify right))
-  )
-  (hierarchical_label "SCL" (shape output) (at 154.94 80.01 0) (fields_autoplaced)
+  (hierarchical_label "Audio_FIL" (shape input) (at 104.14 90.17 180) (fields_autoplaced)
+    (effects (font (size 1.27 1.27)) (justify right))
+  )
+  (hierarchical_label "SCL" (shape output) (at 180.34 109.22 0) (fields_autoplaced)
     (effects (font (size 1.27 1.27)) (justify left))
   )
@@
     )
   )
+  (symbol (lib_id "power:GND") (at 180.34 60.96 0) (unit 1)
+    (in_bom yes) (on_board yes) (dnp no) (fields_autoplaced)
+    (property "Reference" "#PWR039" (at 180.34 67.31 0)
+      (effects (font (size 1.27 1.27)) hide)
+    )
+    (property "Value" "GND" (at 180.34 66.04 0)
+      (effects (font (size 1.27 1.27)))
+    )
+    (property "Footprint" "" (at 180.34 60.96 0)
+      (effects (font (size 1.27 1.27)) hide)
+    )
+    (property "Datasheet" "" (at 180.34 60.96 0)
+      (effects (font (size 1.27 1.27)) hide)
+    )
+    (pin "1")
+    (instances
+      (project "VibeLight"
+        (path "/704dec10-a4c2-4298-be85-193d9407f59f/a98cecf9-ef60-4d48-8d8f-6fc42778f104"
+          (reference "#PWR039") (unit 1)
+        )
+      )
+    )
+  )
   (symbol (lib_id "power:GND") (at 190.5 97.79 0) (unit 1)
     (in_bom yes) (on_board yes) (dnp no) (fields_autoplaced)
@@
         (path "/704dec10-a4c2-4298-be85-193d9407f59f/a98cecf9-ef60-4d48-8d8f-6fc42778f104"
           (reference "#PWR017") (unit 1)
+        )
+      )
+    )
+  )
+  (symbol (lib_id "Connector:Conn_ARM_SWD_TagConnect_TC2030") (at 182.88 50.8 0) (unit 1)
+    (in_bom no) (on_board yes) (dnp no) (fields_autoplaced)
+    (property "Reference" "J1" (at 176.53 49.53 0)
+      (effects (font (size 1.27 1.27)) (justify right))
+    )
+    (property "Value" "Conn_ARM_SWD_TagConnect_TC2030" (at 176.53 52.07 0)
+      (effects (font (size 1.27 1.27)) (justify right))
+    )
+    (property "Footprint" "Connector:Tag-Connect_TC2030-IDC-NL_2x03_P1.27mm_Vertical" (at 182.88 68.58 0)
+      (effects (font (size 1.27 1.27)) hide)
+    )
+    (property "Datasheet" "https://www.tag-connect.com/wp-content/uploads/bsk-pdf-manager/TC2030-CTX_1.pdf" (at 182.88 66.04 0)
+      (effects (font (size 1.27 1.27)) hide)
+    )
+    (pin "1")
+    (pin "2")
+    (pin "3")
+    (pin "4")
+    (pin "5")
+    (pin "6")
+    (instances
+      (project "VibeLight"
+        (path "/704dec10-a4c2-4298-be85-193d9407f59f/a98cecf9-ef60-4d48-8d8f-6fc42778f104"
+          (reference "J1") (unit 1)
         )
       )
@@
         )
       )
+    )
+  )
+  (symbol (lib_id "power:+3V3") (at 180.34 40.64 0) (unit 1)
+    (in_bom yes) (on_board yes) (dnp no) (fields_autoplaced)
+    (property "Reference" "#PWR038" (at 180.34 44.45 0)
+      (effects (font (size 1.27 1.27)) hide)
+    )
+    (property "Value" "+3V3" (at 180.34 35.56 0)
+      (effects (font (size 1.27 1.27)))
+    )
+    (property "Footprint" "" (at 180.34 40.64 0)
+      (effects (font (size 1.27 1.27)) hide)
+    )
+    (property "Datasheet" "" (at 180.34 40.64 0)
+      (effects (font (size 1.27 1.27)) hide)
+    )
+    (pin "1")
+    (instances
+      (project "VibeLight"
+        (path "/704dec10-a4c2-4298-be85-193d9407f59f/a98cecf9-ef60-4d48-8d8f-6fc42778f104"
+          (reference "#PWR038") (unit 1)
+        )
+      )
