File: MCU.kicad_sch (KiCad schematic)
At the start: 3 parts, among them U2 BL652

Commit message: misc changes during call
Connections:
- net RES2: now reaches U2.14 (SIO_10/NFC2)
- net RES: now reaches U2.15 (SIO_09/NFC1)
- net Intensity_dial renamed Intensity_Dial
Changed lines of the file:
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@@
+    (stroke (width 0) (type default))
+  )
+  (wire (pts (xy 101.6 102.87) (xy 104.14 102.87))
     (stroke (width 0) (type default))
   )
@@
   )
   (wire (pts (xy 60.96 87.63) (xy 62.23 87.63))
+    (stroke (width 0) (type default))
+  )
+  (wire (pts (xy 101.6 105.41) (xy 104.14 105.41))
     (stroke (width 0) (type default))
   )
@@
     (effects (font (size 1.27 1.27)) (justify left bottom))
   )
+  (label "RES2" (at 101.6 105.41 0) (fields_autoplaced)
+    (effects (font (size 1.27 1.27)) (justify left bottom))
+  )
+  (label "RES" (at 101.6 102.87 0) (fields_autoplaced)
+    (effects (font (size 1.27 1.27)) (justify left bottom))
+  )
   (global_label "SDA" (shape input) (at 78.74 114.3 180) (fields_autoplaced)
     (effects (font (size 1.27 1.27)) (justify right))
@@
     )
   )
-  (global_label "Intensity_dial" (shape input) (at 95.25 90.17 180) (fields_autoplaced)
-    (effects (font (size 1.27 1.27)) (justify right))
-    (property "Intersheetrefs" "${INTERSHEET_REFS}" (at 79.6859 90.17 0)
-      (effects (font (size 1.27 1.27)) (justify right) hide)
-    )
-  )
   (global_label "SCL" (shape input) (at 78.74 110.49 180) (fields_autoplaced)
     (effects (font (size 1.27 1.27)) (justify right))
@@
     )
   )
-  (global_label "Audio_FIL" (shape input) (at 95.25 85.09 180) (fields_autoplaced)
-    (effects (font (size 1.27 1.27)) (justify right))
-    (property "Intersheetrefs" "${INTERSHEET_REFS}" (at 83.4353 85.09 0)
-      (effects (font (size 1.27 1.27)) (justify right) hide)
-    )
-  )
   (global_label "SW1" (shape input) (at 78.74 99.06 180) (fields_autoplaced)
     (effects (font (size 1.27 1.27)) (justify right))
@@
     )
   )
+  (hierarchical_label "Audio_FIL" (shape input) (at 95.25 85.09 180) (fields_autoplaced)
+    (effects (font (size 1.27 1.27)) (justify right))
+  )
+  (hierarchical_label "Intensity_Dial" (shape input) (at 95.25 90.17 180) (fields_autoplaced)
+    (effects (font (size 1.27 1.27)) (justify right))
+  )
   (symbol (lib_id "Device:R") (at 62.23 91.44 0) (unit 1)

Commit message: started work on pcb layout
started work on pcb layout
Connections:
- net SWCLK is gone; now on net SCL: U2.6 (SWDCLK)
- net SWDIO is gone; now on net SDA: U2.5 (SWDIO)
- net Batt_Meas: now also U2.38 (SIO_25); no longer U2.20 (SIO_05/AIN3)
- net Battery: now also U2.26 (VDD)
- net SW1: now also U2.29 (SIO_15)
- net SW2: now also U2.10 (SIO_16)
- net ACC_INT1: now reaches U2.2 (SIO_24)
- net ACC_INT2: now reaches U2.3 (SIO_23)
- net LED_CNTRL: now reaches U2.36 (SIO_27)
- net OPT_INT: now reaches U2.4 (SIO_22)
Other:
- moved on the sheet: R1, R2
Changed lines of the file:
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@@
   (junction (at 127 128.27) (diameter 0) (color 0 0 0 0)
   )
-  (junction (at 62.23 95.25) (diameter 0) (color 0 0 0 0)
+  (junction (at 60.96 95.25) (diameter 0) (color 0 0 0 0)
   )
   (junction (at 132.08 128.27) (diameter 0) (color 0 0 0 0)
   )
+  (junction (at 57.15 87.63) (diameter 0) (color 0 0 0 0)
+  )
   (junction (at 129.54 128.27) (diameter 0) (color 0 0 0 0)
   )
@@
     (stroke (width 0) (type default))
   )
+  (wire (pts (xy 57.15 74.93) (xy 57.15 87.63))
+    (stroke (width 0) (type default))
+  )
+  (wire (pts (xy 154.94 107.95) (xy 160.02 107.95))
+    (stroke (width 0) (type default))
+  )
+  (wire (pts (xy 99.06 120.65) (xy 104.14 120.65))
+    (stroke (width 0) (type default))
+  )
   (wire (pts (xy 95.25 87.63) (xy 104.14 87.63))
     (stroke (width 0) (type default))
   )
-  (wire (pts (xy 95.25 95.25) (xy 95.25 92.71))
+  (wire (pts (xy 83.82 146.05) (xy 83.82 95.25))
+    (stroke (width 0) (type default))
+  )
+  (wire (pts (xy 154.94 100.33) (xy 160.02 100.33))
+    (stroke (width 0) (type default))
+  )
+  (wire (pts (xy 154.94 113.03) (xy 160.02 113.03))
     (stroke (width 0) (type default))
   )
@@
     (stroke (width 0) (type default))
   )
-  (wire (pts (xy 60.96 87.63) (xy 62.23 87.63))
+  (wire (pts (xy 154.94 110.49) (xy 160.02 110.49))
+    (stroke (width 0) (type default))
+  )
+  (wire (pts (xy 99.06 118.11) (xy 104.14 118.11))
     (stroke (width 0) (type default))
   )
@@
     (stroke (width 0) (type default))
   )
-  (wire (pts (xy 62.23 95.25) (xy 95.25 95.25))
+  (wire (pts (xy 60.96 95.25) (xy 83.82 95.25))
     (stroke (width 0) (type default))
   )
@@
     (stroke (width 0) (type default))
   )
+  (wire (pts (xy 54.61 87.63) (xy 57.15 87.63))
+    (stroke (width 0) (type default))
+  )
   (wire (pts (xy 154.94 80.01) (xy 161.29 80.01))
     (stroke (width 0) (type default))
   )
+  (wire (pts (xy 83.82 146.05) (xy 173.99 146.05))
+    (stroke (width 0) (type default))
+  )
+  (wire (pts (xy 57.15 74.93) (xy 129.54 74.93))
+    (stroke (width 0) (type default))
+  )
+  (wire (pts (xy 154.94 105.41) (xy 173.99 105.41))
+    (stroke (width 0) (type default))
+  )
+  (wire (pts (xy 173.99 105.41) (xy 173.99 146.05))
+    (stroke (width 0) (type default))
+  )
+  (wire (pts (xy 57.15 87.63) (xy 60.96 87.63))
+    (stroke (width 0) (type default))
+  )
   (text "TODO\nPower & Gnd\nProgramming Header\nBypass Caps\n" (at 101.6 63.5 0)
     (effects (font (size 1.27 1.27)) (justify left bottom))
   )
   (text "Battery is 3.3->4.4V\nAnalog input should stay \nunder 1.8V \nso use resistor divider"
-    (at 34.29 99.06 0)
-    (effects (font (size 1.27 1.27)) (justify left bottom))
-  )
-  (label "SWCLK" (at 157.48 80.01 0) (fields_autoplaced)
-    (effects (font (size 1.27 1.27)) (justify left bottom))
-  )
-  (label "SWDIO" (at 157.48 82.55 0) (fields_autoplaced)
-    (effects (font (size 1.27 1.27)) (justify left bottom))
-  )
-  (label "Batt_Meas" (at 71.12 95.25 0) (fields_autoplaced)
+    (at 33.02 99.06 0)
+    (effects (font (size 1.27 1.27)) (justify left bottom))
+  )
+  (label "Batt_Meas" (at 69.85 95.25 0) (fields_autoplaced)
     (effects (font (size 1.27 1.27)) (justify left bottom))
   )
@@
     (effects (font (size 1.27 1.27)) (justify left bottom))
   )
-  (global_label "SDA" (shape input) (at 78.74 114.3 180) (fields_autoplaced)
-    (effects (font (size 1.27 1.27)) (justify right))
-    (property "Intersheetrefs" "${INTERSHEET_REFS}" (at 72.1867 114.3 0)
-      (effects (font (size 1.27 1.27)) (justify right) hide)
-    )
-  )
-  (global_label "SW2" (shape input) (at 78.74 104.14 180) (fields_autoplaced)
-    (effects (font (size 1.27 1.27)) (justify right))
-    (property "Intersheetrefs" "${INTERSHEET_REFS}" (at 71.8844 104.14 0)
-      (effects (font (size 1.27 1.27)) (justify right) hide)
-    )
-  )
-  (global_label "Battery" (shape input) (at 60.96 87.63 180) (fields_autoplaced)
-    (effects (font (size 1.27 1.27)) (justify right))
-    (property "Intersheetrefs" "${INTERSHEET_REFS}" (at 51.262 87.63 0)
-      (effects (font (size 1.27 1.27)) (justify right) hide)
-    )
-  )
-  (global_label "SCL" (shape input) (at 78.74 110.49 180) (fields_autoplaced)
-    (effects (font (size 1.27 1.27)) (justify right))
-    (property "Intersheetrefs" "${INTERSHEET_REFS}" (at 72.2472 110.49 0)
-      (effects (font (size 1.27 1.27)) (justify right) hide)
-    )
-  )
-  (global_label "Audio_RAW" (shape input) (at 95.25 87.63 180) (fields_autoplaced)
-    (effects (font (size 1.27 1.27)) (justify right))
-    (property "Intersheetrefs" "${INTERSHEET_REFS}" (at 82.3468 87.63 0)
-      (effects (font (size 1.27 1.27)) (justify right) hide)
-    )
-  )
-  (global_label "SW1" (shape input) (at 78.74 99.06 180) (fields_autoplaced)
-    (effects (font (size 1.27 1.27)) (justify right))
-    (property "Intersheetrefs" "${INTERSHEET_REFS}" (at 71.8844 99.06 0)
-      (effects (font (size 1.27 1.27)) (justify right) hide)
-    )
+  (hierarchical_label "SW2" (shape input) (at 99.06 120.65 180) (fields_autoplaced)
+    (effects (font (size 1.27 1.27)) (justify right))
+  )
+  (hierarchical_label "Audio_RAW" (shape input) (at 95.25 87.63 180) (fields_autoplaced)
+    (effects (font (size 1.27 1.27)) (justify right))
+  )
+  (hierarchical_label "LED_CNTRL" (shape output) (at 160.02 100.33 0) (fields_autoplaced)
+    (effects (font (size 1.27 1.27)) (justify left))
+  )
+  (hierarchical_label "Battery" (shape input) (at 54.61 87.63 180) (fields_autoplaced)
+    (effects (font (size 1.27 1.27)) (justify right))
+  )
+  (hierarchical_label "OPT_INT" (shape input) (at 160.02 113.03 0) (fields_autoplaced)
+    (effects (font (size 1.27 1.27)) (justify left))
+  )
+  (hierarchical_label "SDA" (shape output) (at 161.29 82.55 0) (fields_autoplaced)
+    (effects (font (size 1.27 1.27)) (justify left))
+  )
+  (hierarchical_label "ACC_INT1" (shape input) (at 160.02 107.95 0) (fields_autoplaced)
+    (effects (font (size 1.27 1.27)) (justify left))
+  )
+  (hierarchical_label "ACC_INT2" (shape input) (at 160.02 110.49 0) (fields_autoplaced)
+    (effects (font (size 1.27 1.27)) (justify left))
+  )
+  (hierarchical_label "SW1" (shape input) (at 99.06 118.11 180) (fields_autoplaced)
+    (effects (font (size 1.27 1.27)) (justify right))
   )
   (hierarchical_label "Audio_FIL" (shape input) (at 95.25 85.09 180) (fields_autoplaced)
     (effects (font (size 1.27 1.27)) (justify right))
   )
+  (hierarchical_label "SCL" (shape output) (at 161.29 80.01 0) (fields_autoplaced)
+    (effects (font (size 1.27 1.27)) (justify left))
+  )
   (hierarchical_label "Intensity_Dial" (shape input) (at 95.25 90.17 180) (fields_autoplaced)
     (effects (font (size 1.27 1.27)) (justify right))
   )
-  (symbol (lib_id "Device:R") (at 62.23 91.44 0) (unit 1)
+  (symbol (lib_id "Device:R") (at 60.96 91.44 0) (unit 1)
     (in_bom yes) (on_board yes) (dnp no) (fields_autoplaced)
-    (property "Reference" "R1" (at 64.77 90.17 0)
-      (effects (font (size 1.27 1.27)) (justify left))
-    )
-    (property "Value" "R" (at 64.77 92.71 0)
-      (effects (font (size 1.27 1.27)) (justify left))
-    )
-    (property "Footprint" "Resistor_SMD:R_0603_1608Metric_Pad0.98x0.95mm_HandSolder" (at 60.452 91.44 90)
-      (effects (font (size 1.27 1.27)) hide)
-    )
-    (property "Datasheet" "~" (at 62.23 91.44 0)
+    (property "Reference" "R1" (at 63.5 90.17 0)
+      (effects (font (size 1.27 1.27)) (justify left))
+    )
+    (property "Value" "R" (at 63.5 92.71 0)
+      (effects (font (size 1.27 1.27)) (justify left))
+    )
+    (property "Footprint" "Resistor_SMD:R_0603_1608Metric_Pad0.98x0.95mm_HandSolder" (at 59.182 91.44 90)
+      (effects (font (size 1.27 1.27)) hide)
+    )
+    (property "Datasheet" "~" (at 60.96 91.44 0)
       (effects (font (size 1.27 1.27)) hide)
     )
@@
     )
   )
-  (symbol (lib_id "power:GND") (at 62.23 102.87 0) (unit 1)
+  (symbol (lib_id "power:GND") (at 60.96 102.87 0) (unit 1)
     (in_bom yes) (on_board yes) (dnp no) (fields_autoplaced)
-    (property "Reference" "#PWR09" (at 62.23 109.22 0)
-      (effects (font (size 1.27 1.27)) hide)
-    )
-    (property "Value" "GND" (at 62.23 107.95 0)
+    (property "Reference" "#PWR09" (at 60.96 109.22 0)
+      (effects (font (size 1.27 1.27)) hide)
+    )
+    (property "Value" "GND" (at 60.96 107.95 0)
       (effects (font (size 1.27 1.27)))
     )
-    (property "Footprint" "" (at 62.23 102.87 0)
-      (effects (font (size 1.27 1.27)) hide)
-    )
-    (property "Datasheet" "" (at 62.23 102.87 0)
+    (property "Footprint" "" (at 60.96 102.87 0)
+      (effects (font (size 1.27 1.27)) hide)
+    )
+    (property "Datasheet" "" (at 60.96 102.87 0)
       (effects (font (size 1.27 1.27)) hide)
     )
@@
     )
   )
-  (symbol (lib_id "Device:R") (at 62.23 99.06 0) (unit 1)
+  (symbol (lib_id "Device:R") (at 60.96 99.06 0) (unit 1)
     (in_bom yes) (on_board yes) (dnp no) (fields_autoplaced)
-    (property "Reference" "R2" (at 64.77 97.79 0)
-      (effects (font (size 1.27 1.27)) (justify left))
-    )
-    (property "Value" "R" (at 64.77 100.33 0)
-      (effects (font (size 1.27 1.27)) (justify left))
-    )
-    (property "Footprint" "Resistor_SMD:R_0603_1608Metric_Pad0.98x0.95mm_HandSolder" (at 60.452 99.06 90)
-      (effects (font (size 1.27 1.27)) hide)
-    )
-    (property "Datasheet" "~" (at 62.23 99.06 0)
-      (effects (font (size 1.27 1.27)) hide)
-    )
+    (property "Reference" "R2" (at 63.5 97.79 0)
+      (effects (font (size 1.27 1.27)) (justify left))
+    )
+    (property "Value" "R" (at 63.5 100.33 0)
+      (effects (font (size 1.27 1.27)) (justify left))
+    )
+    (property "Footprint" "Resistor_SMD:R_0603_1608Metric_Pad0.98x0.95mm_HandSolder" (at 59.182 99.06 90)
+      (effects (font (size 1.27 1.27)) hide)
+    )
+    (property "Datasheet" "~" (at 60.96 99.06 0)
+      (effects (font (size 1.27 1.27)) hide)
+    )

Commit message: completed rev1 of PCB layout
need to double check components and other elements, connections, and add values
Connections:
- net ACC_INT1: now also U2.17 (SIO_08); no longer U2.2 (SIO_24)
- net ACC_INT2: now also U2.18 (SIO_07); no longer U2.3 (SIO_23)
- net Intensity_Dial: now also U2.4 (SIO_22); no longer U2.21 (SIO_04/AIN2)
- net LED_CNTRL: no longer U2.36 (SIO_27)
- net OPT_INT: now also U2.19 (SIO_06); no longer U2.4 (SIO_22)
- net SW1: now also U2.2 (SIO_24); no longer U2.29 (SIO_15)
- net SW2: now also U2.3 (SIO_23); no longer U2.10 (SIO_16)
Changed lines of the file:
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@@
-    (stroke (width 0) (type default))
-  )
-  (wire (pts (xy 154.94 107.95) (xy 160.02 107.95))
-    (stroke (width 0) (type default))
-  )
-  (wire (pts (xy 99.06 120.65) (xy 104.14 120.65))
-    (stroke (width 0) (type default))
-  )
-  (wire (pts (xy 95.25 87.63) (xy 104.14 87.63))
     (stroke (width 0) (type default))
   )
@@
     (stroke (width 0) (type default))
   )
-  (wire (pts (xy 154.94 100.33) (xy 160.02 100.33))
-    (stroke (width 0) (type default))
-  )
-  (wire (pts (xy 154.94 113.03) (xy 160.02 113.03))
-    (stroke (width 0) (type default))
-  )
   (wire (pts (xy 101.6 102.87) (xy 104.14 102.87))
-    (stroke (width 0) (type default))
-  )
-  (wire (pts (xy 95.25 90.17) (xy 104.14 90.17))
-    (stroke (width 0) (type default))
-  )
-  (wire (pts (xy 154.94 82.55) (xy 161.29 82.55))
-    (stroke (width 0) (type default))
-  )
-  (wire (pts (xy 154.94 110.49) (xy 160.02 110.49))
-    (stroke (width 0) (type default))
-  )
-  (wire (pts (xy 99.06 118.11) (xy 104.14 118.11))
     (stroke (width 0) (type default))
   )
@@
     (stroke (width 0) (type default))
   )
-  (wire (pts (xy 95.25 92.71) (xy 104.14 92.71))
-    (stroke (width 0) (type default))
-  )
-  (wire (pts (xy 95.25 85.09) (xy 104.14 85.09))
-    (stroke (width 0) (type default))
-  )
   (wire (pts (xy 54.61 87.63) (xy 57.15 87.63))
-    (stroke (width 0) (type default))
-  )
-  (wire (pts (xy 154.94 80.01) (xy 161.29 80.01))
     (stroke (width 0) (type default))
   )
@@
     (effects (font (size 1.27 1.27)) (justify left bottom))
   )
-  (hierarchical_label "SW2" (shape input) (at 99.06 120.65 180) (fields_autoplaced)
-    (effects (font (size 1.27 1.27)) (justify right))
+  (hierarchical_label "SW2" (shape input) (at 154.94 110.49 0) (fields_autoplaced)
+    (effects (font (size 1.27 1.27)) (justify left))
   )
-  (hierarchical_label "Audio_RAW" (shape input) (at 95.25 87.63 180) (fields_autoplaced)
+  (hierarchical_label "Audio_RAW" (shape input) (at 104.14 87.63 180) (fields_autoplaced)
     (effects (font (size 1.27 1.27)) (justify right))
   )
@@
     (effects (font (size 1.27 1.27)) (justify right))
   )
-  (hierarchical_label "OPT_INT" (shape input) (at 160.02 113.03 0) (fields_autoplaced)
+  (hierarchical_label "OPT_INT" (shape input) (at 104.14 95.25 180) (fields_autoplaced)
+    (effects (font (size 1.27 1.27)) (justify right))
+  )
+  (hierarchical_label "SDA" (shape output) (at 154.94 82.55 0) (fields_autoplaced)
     (effects (font (size 1.27 1.27)) (justify left))
   )
-  (hierarchical_label "SDA" (shape output) (at 161.29 82.55 0) (fields_autoplaced)
+  (hierarchical_label "ACC_INT1" (shape input) (at 104.14 100.33 180) (fields_autoplaced)
+    (effects (font (size 1.27 1.27)) (justify right))
+  )
+  (hierarchical_label "ACC_INT2" (shape input) (at 104.14 97.79 180) (fields_autoplaced)
+    (effects (font (size 1.27 1.27)) (justify right))
+  )
+  (hierarchical_label "SW1" (shape input) (at 154.94 107.95 0) (fields_autoplaced)
     (effects (font (size 1.27 1.27)) (justify left))
   )
-  (hierarchical_label "ACC_INT1" (shape input) (at 160.02 107.95 0) (fields_autoplaced)
+  (hierarchical_label "Audio_FIL" (shape input) (at 104.14 85.09 180) (fields_autoplaced)
+    (effects (font (size 1.27 1.27)) (justify right))
+  )
+  (hierarchical_label "SCL" (shape output) (at 154.94 80.01 0) (fields_autoplaced)
     (effects (font (size 1.27 1.27)) (justify left))
   )
-  (hierarchical_label "ACC_INT2" (shape input) (at 160.02 110.49 0) (fields_autoplaced)
+  (hierarchical_label "Intensity_Dial" (shape input) (at 154.94 113.03 0) (fields_autoplaced)
     (effects (font (size 1.27 1.27)) (justify left))
   )
-  (hierarchical_label "SW1" (shape input) (at 99.06 118.11 180) (fields_autoplaced)
-    (effects (font (size 1.27 1.27)) (justify right))
-  )
-  (hierarchical_label "Audio_FIL" (shape input) (at 95.25 85.09 180) (fields_autoplaced)
-    (effects (font (size 1.27 1.27)) (justify right))
-  )
-  (hierarchical_label "SCL" (shape output) (at 161.29 80.01 0) (fields_autoplaced)
-    (effects (font (size 1.27 1.27)) (justify left))
-  )
-  (hierarchical_label "Intensity_Dial" (shape input) (at 95.25 90.17 180) (fields_autoplaced)
-    (effects (font (size 1.27 1.27)) (justify right))
-  )
   (symbol (lib_id "Device:R") (at 60.96 91.44 0) (unit 1)

Commit message: Changes from DR call
Parts:
- added C4: 100nF, Capacitor_SMD:C_0603_1608Metric_Pad1.08x0.95mm_HandSolder, symbol Device:C
Connections:
- net Battery: no longer U2.26 (VDD)
- net GND: now also C4.2
- new net +3V3: C4.1, U2.26 (VDD)
Changed lines of the file:
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@@
   (junction (at 60.96 95.25) (diameter 0) (color 0 0 0 0)
   )
+  (junction (at 129.54 67.31) (diameter 0) (color 0 0 0 0)
+  )
   (junction (at 132.08 128.27) (diameter 0) (color 0 0 0 0)
   )
-  (junction (at 57.15 87.63) (diameter 0) (color 0 0 0 0)
-  )
   (junction (at 129.54 128.27) (diameter 0) (color 0 0 0 0)
   )
@@
     (stroke (width 0) (type default))
   )
-  (wire (pts (xy 57.15 74.93) (xy 57.15 87.63))
-    (stroke (width 0) (type default))
-  )
   (wire (pts (xy 83.82 146.05) (xy 83.82 95.25))
     (stroke (width 0) (type default))
   )
+  (wire (pts (xy 129.54 67.31) (xy 129.54 74.93))
+    (stroke (width 0) (type default))
+  )
   (wire (pts (xy 101.6 102.87) (xy 104.14 102.87))
     (stroke (width 0) (type default))
@@
     (stroke (width 0) (type default))
   )
-  (wire (pts (xy 54.61 87.63) (xy 57.15 87.63))
+  (wire (pts (xy 129.54 67.31) (xy 142.24 67.31))
     (stroke (width 0) (type default))
   )
@@
     (stroke (width 0) (type default))
   )
-  (wire (pts (xy 57.15 74.93) (xy 129.54 74.93))
-    (stroke (width 0) (type default))
-  )
   (wire (pts (xy 154.94 105.41) (xy 173.99 105.41))
     (stroke (width 0) (type default))
@@
     (stroke (width 0) (type default))
   )
-  (wire (pts (xy 57.15 87.63) (xy 60.96 87.63))
+  (wire (pts (xy 54.61 87.63) (xy 60.96 87.63))
+    (stroke (width 0) (type default))
+  )
+  (wire (pts (xy 129.54 59.69) (xy 129.54 67.31))
     (stroke (width 0) (type default))
   )
@@
     )
   )
+  (symbol (lib_id "Device:C") (at 142.24 71.12 0) (unit 1)
+    (in_bom yes) (on_board yes) (dnp no) (fields_autoplaced)
+    (property "Reference" "C4" (at 146.05 69.85 0)
+      (effects (font (size 1.27 1.27)) (justify left))
+    )
+    (property "Value" "100nF" (at 146.05 72.39 0)
+      (effects (font (size 1.27 1.27)) (justify left))
+    )
+    (property "Footprint" "Capacitor_SMD:C_0603_1608Metric_Pad1.08x0.95mm_HandSolder" (at 143.2052 74.93 0)
+      (effects (font (size 1.27 1.27)) hide)
+    )
+    (property "Datasheet" "~" (at 142.24 71.12 0)
+      (effects (font (size 1.27 1.27)) hide)
+    )
+    (pin "1")
+    (pin "2")
+    (instances
+      (project "VibeLight"
+        (path "/704dec10-a4c2-4298-be85-193d9407f59f"
+          (reference "C4") (unit 1)
+        )
+        (path "/704dec10-a4c2-4298-be85-193d9407f59f/a98cecf9-ef60-4d48-8d8f-6fc42778f104"
+          (reference "C8") (unit 1)
+        )
+      )
+    )
+  )
   (symbol (lib_id "power:GND") (at 60.96 102.87 0) (unit 1)
     (in_bom yes) (on_board yes) (dnp no) (fields_autoplaced)
@@
     )
   )
+  (symbol (lib_id "power:+3V3") (at 129.54 59.69 0) (unit 1)
+    (in_bom yes) (on_board yes) (dnp no) (fields_autoplaced)
+    (property "Reference" "#PWR017" (at 129.54 63.5 0)
+      (effects (font (size 1.27 1.27)) hide)
+    )
+    (property "Value" "+3V3" (at 129.54 54.61 0)
+      (effects (font (size 1.27 1.27)))
+    )
+    (property "Footprint" "" (at 129.54 59.69 0)
+      (effects (font (size 1.27 1.27)) hide)
+    )
+    (property "Datasheet" "" (at 129.54 59.69 0)
+      (effects (font (size 1.27 1.27)) hide)
+    )
+    (pin "1")
+    (instances
+      (project "VibeLight"
+        (path "/704dec10-a4c2-4298-be85-193d9407f59f/a98cecf9-ef60-4d48-8d8f-6fc42778f104"
+          (reference "#PWR017") (unit 1)
+        )
+      )
+    )
+  )
   (symbol (lib_id "Device:R") (at 60.96 99.06 0) (unit 1)
     (in_bom yes) (on_board yes) (dnp no) (fields_autoplaced)
@@
         )
       )
+    )
+  )
+  (symbol (lib_id "power:GND") (at 142.24 74.93 0) (unit 1)
+    (in_bom yes) (on_board yes) (dnp no) (fields_autoplaced)
+    (property "Reference" "#PWR023" (at 142.24 81.28 0)
+      (effects (font (size 1.27 1.27)) hide)
+    )
+    (property "Value" "GND" (at 142.24 80.01 0)
+      (effects (font (size 1.27 1.27)))
+    )
+    (property "Footprint" "" (at 142.24 74.93 0)
+      (effects (font (size 1.27 1.27)) hide)
+    )
+    (property "Datasheet" "" (at 142.24 74.93 0)
+      (effects (font (size 1.27 1.27)) hide)
+    )
+    (pin "1")
+    (instances
+      (project "VibeLight"
+        (path "/704dec10-a4c2-4298-be85-193d9407f59f/a98cecf9-ef60-4d48-8d8f-6fc42778f104"
+          (reference "#PWR023") (unit 1)
+        )
+      )
