File: VibeLight.kicad_pcb (KiCad board)
At the start: 2 copper layers, 31.5 x 34 mm, 36 parts, among them SW1 SW_Push, SW2 SW_Push, U2 SPV08A0LR5H-1, U3 BL652

Commit message: updates from call
Parts:
- added J1: Conn_ARM_SWD_TagConnect_TC2030, Connector:Tag-Connect_TC2030-IDC-NL_2x03_P1.27mm_Vertical, B.Cu at (22.3, 21.3)
- added R5: 100, Resistor_SMD:R_0603_1608Metric_Pad0.98x0.95mm_HandSolder, F.Cu at (24.0, 48.6)
- moved SW1 33.8 mm to (52.6, 33.8)
- moved SW2 29.9 mm to (52.3, 37.9)
- turned C2 to 0 degrees
Connections:
- D2 pad 1: GND -> Net-(D2-K)
- D2 pad 2: /MCU/BATT_LVL -> +3V3
- R1 pad 2: Net-(U3-SIO_26) -> Net-(U3-SIO_28/AIN4)
- R2 pad 1: Net-(U3-SIO_26) -> Net-(U3-SIO_28/AIN4)
- U3 pad 21: unconnected-(U3-SIO_04/AIN2-Pad21) -> /Audio Input/FIL
- U3 pad 23: /Audio Input/FIL -> unconnected-(U3-SIO_02/AIN0-Pad23)
- U3 pad 35: unconnected-(U3-SIO_28/AIN4-Pad35) -> Net-(U3-SIO_28/AIN4)
- U3 pad 37: Net-(U3-SIO_26) -> unconnected-(U3-SIO_26-Pad37)
- U3 pad 5: /SDA -> /MCU/SWD
- U3 pad 6: /SCL -> /MCU/SWCLK
Routing:
- net /MCU/BATT_LVL: track 17.4 -> 0.00 mm, vias 2 -> 0
- net +3V3: track 106.4 -> 98.2 mm, vias 0 -> 2
- net /SCL: track 53.7 -> 46.7 mm
- net GND: track 3.20 -> 9.23 mm, vias 0 -> 20
- net Net-(U3-SIO_26): track 4.89 -> 0.00 mm
- net Net-(U3-SIO_28/AIN4): track 0.00 -> 4.27 mm
- net /SDA: track 53.1 -> 50.9 mm, vias 6 -> 5
- net /Audio Input/FIL: track 23.2 -> 22.7 mm, vias 2 -> 0
- net /Audio Input/RAW: track 27.5 -> 27.0 mm, vias 4 -> 2
- net /MCU/ACC_INT1: vias 2 -> 0
- net /MCU/OPT_INT: vias 2 -> 0
- net /MCU/ACC_INT2: vias 2 -> 0
