File: audio_input.kicad_sch (KiCad schematic)
At the start: 14 parts

Commit message: updates from call
Parts:
- added U1: MCP6002-xMC, Package_DFN_QFN:DFN-8-1EP_3x2mm_P0.5mm_EP1.75x1.45mm, symbol Amplifier_Operational:MCP6002-xMC
Connections:
- new net: U1.4 (V-), U1.9 (V-)
Changed lines of the file:
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@@
+    )
+  )
+  (symbol (lib_id "Amplifier_Operational:MCP6002-xMC") (at 67.31 59.69 0) (unit 3)
+    (in_bom yes) (on_board yes) (dnp no) (fields_autoplaced)
+    (property "Reference" "U1" (at 66.04 58.42 0)
+      (effects (font (size 1.27 1.27)) (justify left))
+    )
+    (property "Value" "MCP6002-xMC" (at 66.04 60.96 0)
+      (effects (font (size 1.27 1.27)) (justify left))
+    )
+    (property "Footprint" "Package_DFN_QFN:DFN-8-1EP_3x2mm_P0.5mm_EP1.75x1.45mm" (at 67.31 59.69 0)
+      (effects (font (size 1.27 1.27)) hide)
+    )
+    (property "Datasheet" "http://ww1.microchip.com/downloads/en/DeviceDoc/21733j.pdf" (at 67.31 59.69 0)
+      (effects (font (size 1.27 1.27)) hide)
+    )
+    (pin "1")
+    (pin "2")
+    (pin "3")
+    (pin "5")
+    (pin "6")
+    (pin "7")
+    (pin "4")
+    (pin "8")
+    (pin "9")
+    (instances
+      (project "VibeLight"
+        (path "/704dec10-a4c2-4298-be85-193d9407f59f/964563b4-99e1-4b3d-857d-35f5fde5aa09"
+          (reference "U1") (unit 3)
+        )
+      )
+    )
+  )
+  (symbol (lib_id "Amplifier_Operational:MCP6002-xMC") (at 49.53 72.39 0) (unit 2)
+    (in_bom yes) (on_board yes) (dnp no) (fields_autoplaced)
+    (property "Reference" "U1" (at 49.53 62.23 0)
+      (effects (font (size 1.27 1.27)))
+    )
+    (property "Value" "MCP6002-xMC" (at 49.53 64.77 0)
+      (effects (font (size 1.27 1.27)))
+    )
+    (property "Footprint" "Package_DFN_QFN:DFN-8-1EP_3x2mm_P0.5mm_EP1.75x1.45mm" (at 49.53 72.39 0)
+      (effects (font (size 1.27 1.27)) hide)
+    )
+    (property "Datasheet" "http://ww1.microchip.com/downloads/en/DeviceDoc/21733j.pdf" (at 49.53 72.39 0)
+      (effects (font (size 1.27 1.27)) hide)
+    )
+    (pin "1")
+    (pin "2")
+    (pin "3")
+    (pin "5")
+    (pin "6")
+    (pin "7")
+    (pin "4")
+    (pin "8")
+    (pin "9")
+    (instances
+      (project "VibeLight"
+        (path "/704dec10-a4c2-4298-be85-193d9407f59f/964563b4-99e1-4b3d-857d-35f5fde5aa09"
+          (reference "U1") (unit 2)
+        )
+      )
     )
   )
@@
         )
       )
+    )
+  )
+  (symbol (lib_id "Amplifier_Operational:MCP6002-xMC") (at 49.53 55.88 0) (unit 1)
+    (in_bom yes) (on_board yes) (dnp no) (fields_autoplaced)
+    (property "Reference" "U1" (at 49.53 45.72 0)
+      (effects (font (size 1.27 1.27)))
+    )
+    (property "Value" "MCP6002-xMC" (at 49.53 48.26 0)
+      (effects (font (size 1.27 1.27)))
+    )
+    (property "Footprint" "Package_DFN_QFN:DFN-8-1EP_3x2mm_P0.5mm_EP1.75x1.45mm" (at 49.53 55.88 0)
+      (effects (font (size 1.27 1.27)) hide)
+    )
+    (property "Datasheet" "http://ww1.microchip.com/downloads/en/DeviceDoc/21733j.pdf" (at 49.53 55.88 0)
+      (effects (font (size 1.27 1.27)) hide)
+    )
+    (pin "1")
+    (pin "2")
+    (pin "3")
+    (pin "5")
+    (pin "6")
+    (pin "7")
+    (pin "4")
+    (pin "8")
+    (pin "9")
+    (instances
+      (project "VibeLight"
+        (path "/704dec10-a4c2-4298-be85-193d9407f59f/964563b4-99e1-4b3d-857d-35f5fde5aa09"
+          (reference "U1") (unit 1)
+        )
+      )
