File: audio_input.kicad_sch (KiCad schematic)
At the start: 16 parts

Commit message: updated resistor value in audio filter
Parts:
- Re1: value 620R -> 634R
Changed lines of the file:
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@@
       (effects (font (size 1.27 1.27)))
     )
-    (property "Value" "620R" (at 173.99 87.63 90)
+    (property "Value" "634R" (at 173.99 87.63 90)
       (effects (font (size 1.27 1.27)))
     )
