File: VibeLight.kicad_sch (KiCad schematic)
At the start: 17 parts, among them SW1 SW_Push, SW2 SW_Push

Commit message: new pcb rev with updated audio filter
The only ERC and DRC warnings/errors are unconnected pins and silkscreen text issues. There are two DRC issues that have to do with the mic, but I don't think they're an issue
Parts:
- removed D2: LED, LED_SMD:LED_0603_1608Metric_Pad1.05x0.95mm_HandSolder, symbol Device:LED
- renumbered Accel1 to ACCEL1, OUT_PINS1 to LED_OUT1, Light1 to LIGHT1, PWR_IN1 to PWR1, PWR_REG1 to REG1, Temp1 to TEMP1
Other:
- sheet MCU ports: added none; removed BATT_LVL
Changed lines of the file:
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@@
-    (stroke (width 0) (type default))
-  )
-  (wire (pts (xy 106.68 104.14) (xy 115.57 104.14))
     (stroke (width 0) (type default))
   )
@@
     (stroke (width 0) (type default))
   )
-  (wire (pts (xy 99.06 104.14) (xy 91.44 104.14))
-    (stroke (width 0) (type default))
-  )
   (wire (pts (xy 30.48 109.22) (xy 27.94 109.22))
     (stroke (width 0) (type default))
@@
   )
   (wire (pts (xy 130.81 78.74) (xy 128.27 78.74))
-    (stroke (width 0) (type default))
-  )
-  (wire (pts (xy 91.44 104.14) (xy 91.44 105.41))
     (stroke (width 0) (type default))
   )
@@
   (symbol (lib_id "Connector:Conn_01x03_Pin") (at 27.94 172.72 0) (unit 1)
     (in_bom yes) (on_board yes) (dnp no) (fields_autoplaced)
-    (property "Reference" "OUT_PINS1" (at 28.575 165.1 0)
+    (property "Reference" "LED_OUT1" (at 28.575 165.1 0)
       (effects (font (size 1.27 1.27)))
     )
@@
       (project "VibeLight"
         (path "/704dec10-a4c2-4298-be85-193d9407f59f"
-          (reference "OUT_PINS1") (unit 1)
+          (reference "LED_OUT1") (unit 1)
         )
       )
@@
   (symbol (lib_id "Sensor_Humidity:SHT4x") (at 105.41 73.66 90) (unit 1)
     (in_bom yes) (on_board yes) (dnp no) (fields_autoplaced)
-    (property "Reference" "Temp1" (at 105.41 63.5 90)
+    (property "Reference" "TEMP1" (at 105.41 63.5 90)
       (effects (font (size 1.27 1.27)))
     )
@@
       (project "VibeLight"
         (path "/704dec10-a4c2-4298-be85-193d9407f59f"
-          (reference "Temp1") (unit 1)
+          (reference "TEMP1") (unit 1)
         )
       )
@@
         (path "/704dec10-a4c2-4298-be85-193d9407f59f"
           (reference "#PWR014") (unit 1)
-        )
-      )
-    )
-  )
-  (symbol (lib_id "Device:LED") (at 102.87 104.14 0) (unit 1)
-    (in_bom yes) (on_board yes) (dnp no) (fields_autoplaced)
-    (property "Reference" "D2" (at 101.2825 97.79 0)
-      (effects (font (size 1.27 1.27)))
-    )
-    (property "Value" "LED" (at 101.2825 100.33 0)
-      (effects (font (size 1.27 1.27)))
-    )
-    (property "Footprint" "LED_SMD:LED_0603_1608Metric_Pad1.05x0.95mm_HandSolder" (at 102.87 104.14 0)
-      (effects (font (size 1.27 1.27)) hide)
-    )
-    (property "Datasheet" "~" (at 102.87 104.14 0)
-      (effects (font (size 1.27 1.27)) hide)
-    )
-    (pin "1")
-    (pin "2")
-    (instances
-      (project "VibeLight"
-        (path "/704dec10-a4c2-4298-be85-193d9407f59f"
-          (reference "D2") (unit 1)
         )
       )
@@
   (symbol (lib_id "Sensor_Motion:ADXL343") (at 168.91 74.93 0) (unit 1)
     (in_bom yes) (on_board yes) (dnp no) (fields_autoplaced)
-    (property "Reference" "Accel1" (at 184.15 68.0019 0)
+    (property "Reference" "ACCEL1" (at 184.15 68.0019 0)
       (effects (font (size 1.27 1.27)))
     )
@@
       (project "VibeLight"
         (path "/704dec10-a4c2-4298-be85-193d9407f59f"
-          (reference "Accel1") (unit 1)
+          (reference "ACCEL1") (unit 1)
         )
       )
@@
     )
   )
-  (symbol (lib_id "power:GND") (at 91.44 105.41 0) (unit 1)
-    (in_bom yes) (on_board yes) (dnp no) (fields_autoplaced)
-    (property "Reference" "#PWR037" (at 91.44 111.76 0)
-      (effects (font (size 1.27 1.27)) hide)
-    )
-    (property "Value" "GND" (at 93.98 106.68 0)
-      (effects (font (size 1.27 1.27)) (justify left))
-    )
-    (property "Footprint" "" (at 91.44 105.41 0)
-      (effects (font (size 1.27 1.27)) hide)
-    )
-    (property "Datasheet" "" (at 91.44 105.41 0)
-      (effects (font (size 1.27 1.27)) hide)
-    )
-    (pin "1")
-    (instances
-      (project "VibeLight"
-        (path "/704dec10-a4c2-4298-be85-193d9407f59f"
-          (reference "#PWR037") (unit 1)
-        )
-      )
-    )
-  )
   (symbol (lib_id "power:GND") (at 199.39 107.95 180) (unit 1)
     (in_bom yes) (on_board yes) (dnp no) (fields_autoplaced)
@@
   (symbol (lib_id "Regulator_Linear:LK112M33TR") (at 40.64 109.22 0) (unit 1)
     (in_bom yes) (on_board yes) (dnp no) (fields_autoplaced)
-    (property "Reference" "PWR_REG1" (at 40.64 100.33 0)
+    (property "Reference" "REG1" (at 40.64 100.33 0)
       (effects (font (size 1.27 1.27)))
     )
@@
       (project "VibeLight"
         (path "/704dec10-a4c2-4298-be85-193d9407f59f"
-          (reference "PWR_REG1") (unit 1)
+          (reference "REG1") (unit 1)
         )
       )
@@
   (symbol (lib_id "Connector_Generic:Conn_01x02") (at 26.67 147.32 180) (unit 1)
     (in_bom yes) (on_board yes) (dnp no) (fields_autoplaced)
-    (property "Reference" "PWR_IN1" (at 26.67 138.43 0)
+    (property "Reference" "PWR1" (at 26.67 138.43 0)
       (effects (font (size 1.27 1.27)))
     )
@@
       (project "VibeLight"
         (path "/704dec10-a4c2-4298-be85-193d9407f59f"
-          (reference "PWR_IN1") (unit 1)
+          (reference "PWR1") (unit 1)
         )
       )
@@
   (symbol (lib_name "OPT3002-ALS_1") (lib_id "Sensor_Optical:OPT3002-ALS") (at 212.09 113.03 0) (unit 1)
     (in_bom yes) (on_board yes) (dnp no) (fields_autoplaced)
-    (property "Reference" "Light1" (at 214.1094 91.44 0)
+    (property "Reference" "LIGHT1" (at 214.1094 91.44 0)
       (effects (font (size 1.27 1.27)) (justify left))
     )
@@
       (project "VibeLight"
         (path "/704dec10-a4c2-4298-be85-193d9407f59f"
-          (reference "Light1") (unit 1)
+          (reference "LIGHT1") (unit 1)
         )
       )
@@
       (effects (font (size 1.27 1.27)) (justify right))
     )
-    (pin "BATT_LVL" output (at 115.57 104.14 180)
-      (effects (font (size 1.27 1.27)) (justify left))
-    )
-    (instances
+    (instances
