File: VibeLight.kicad_sch (KiCad schematic)
At the start: 16 parts, among them SW1 SW_Push, SW2 SW_Push

Commit message: Misc updates and tweak. Work still needed, letf notes in top schematic page
Other:
- note added: "Layout notes: need to add programming header Move intensity dial to other side b/c of analog pin locations? I added keepout under the BLE antenna Spind D2 to make routing cleaner, and the change which resistor goes where on MCU for tighter routing There were a few unconnected (ratsnested) grounds that i moved around some components to resolve move the battery resistor divider a bit to get via awa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"
- note added: "Steve Checked (done) Power (done) SHT40 (done) OP3002 (done) Accel MCU Errors: Intensity Dial needs to be analog input Audio Raw and Filter need to be analog inputs Re-Added programming header Mic : Not enough info t give useful feedback overall Recommmend moving LED to before the final filter but not certain I'm guessing you don't want C9 and C12 since you'll actually want the DC component, but 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"
Changed lines of the file:
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@@
     (stroke (width 0) (type default))
+  )
+  (text "Steve Checked\n(done) Power\n(done) SHT40\n(done) OP3002\n(done) Accel\nMCU Errors: \n	Intensity Dial needs to be analog input\n	Audio Raw and Filter need to be analog inputs\n	Re-Added programming header\nMic : \n	Not enough info t give useful feedback overall\n	Recommmend moving LED to before the final filter but not certain \n	I'm guessing you don't want C9 and C12 since you'll actually want the DC component, but it's easy to short them out later so leave them in"
+    (at 25.4 31.75 0)
+    (effects (font (size 1.27 1.27)) (justify left bottom))
+  )
+  (text "Layout notes:\nneed to add programming header\nMove intensity dial to other side b/c of analog pin locations? \nI added keepout under the BLE antenna\nSpind D2 to make routing cleaner, and the change which resistor goes where on MCU for tighter routing\nThere were a few unconnected (ratsnested) grounds that i moved around some components to resolve\nmove the battery resistor divider a bit to get via away from corner\nspun some component groups around to make layout a bit cleaner"
+    (at 20.32 49.53 0)
+    (effects (font (size 1.27 1.27)) (justify left bottom))
   )
   (label "SCL" (at 121.92 91.44 0) (fields_autoplaced)
